File: tt_photometer/tt_photometer.kicad_pcb (KiCad board)
At the start: 2 copper layers, 4 parts, among them J1 Conn_01x03_Male, U1 opt101

Commit message: update
Other:
- board outline added: 16.5 x 29.2 mm
Changed lines of the file:
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@@
   (general
     (thickness 1.6)
-    (drawings 4)
+    (drawings 8)
     (tracks 22)
     (zones 0)
@@
       (outputformat 1)
       (mirror false)
-      (drillshape 1)
+      (drillshape 0)
       (scaleselection 1)
-      (outputdirectory ""))
+      (outputdirectory "gerbers"))
   )
   (net 0 "")
@@
     )
   )
+  (gr_line (start 166.37 67.31) (end 149.86 67.31) (layer Edge.Cuts) (width 0.15))
+  (gr_line (start 166.37 96.52) (end 166.37 67.31) (layer Edge.Cuts) (width 0.15))
+  (gr_line (start 149.86 96.52) (end 166.37 96.52) (layer Edge.Cuts) (width 0.15))
+  (gr_line (start 149.86 67.31) (end 149.86 96.52) (layer Edge.Cuts) (width 0.15))
   (gr_line (start 149.86 67.31) (end 166.37 67.31) (layer B.SilkS) (width 0.2))
   (gr_line (start 166.37 96.52) (end 166.37 67.31) (layer B.SilkS) (width 0.2))
