File: hardware/pcb/tt_nano_HAT_b1/tt_nano_HAT_b1.sch (KiCad schematic (older format))
At the start: 19 parts, among them J1 Conn_01x04_Male, J10 Conn_01x06_Male, J2 Conn_01x06_Male, J3 Conn_01x04_Female, J4 Conn_01x03_Male, J5 Conn_01x03_Male, J6 Conn_01x03_Male, J7 Conn_01x03_Male, J8 Conn_01x03_Male, J9 Conn_01x03_Male

Commit message: Included BOM
Parts:
- added J11: Conn_01x02_Male, Connector_PinHeader_2.54mm:PinHeader_1x02_P2.54mm_Vertical, symbol Connector:Conn_01x02_Male
Connections:
- wire segments 122 -> 127
Changed lines of the file:
@@
 EESchema Schematic File Version 4
-LIBS:tt_nano_HAT-cache
+LIBS:tt_nano_HAT_b1-cache
 EELAYER 26 0
 EELAYER END
@@
 encoding utf-8
 Sheet 1 1
-Title "Test tube photometer"
-Date "2018-11-13"
-Rev "0.1.1"
+Title "Test Tube Photometer"
+Date "2019-03-21"
+Rev "1.1"
 Comp ""
 Comment1 ""
@@
 Connection ~ 3700 1950
 Wire Wire Line
-	3700 1550 3700 1150
+	3700 1550 3700 1300
 Wire Wire Line
 	3700 1150 3800 1150
@@
 	2400 4000 2500 4000
 Connection ~ 2500 4000
+$Comp
+L Connector:Conn_01x02_Male J11
+U 1 1 5C942AC0
+P 2450 1000
+F 0 "J11" H 2556 1178 50  0000 C CNN
+F 1 "Conn_01x02_Male" H 2556 1087 50  0000 C CNN
+F 2 "Connector_PinHeader_2.54mm:PinHeader_1x02_P2.54mm_Vertical" H 2450 1000 50  0001 C CNN
+F 3 "~" H 2450 1000 50  0001 C CNN
+	1    2450 1000
+	1    0    0    -1
+$EndComp
+Wire Wire Line
+	2650 1300 2650 1100
+Wire Wire Line
+	2650 1000 3150 1000
+Wire Wire Line
+	3150 1000 3150 1300
+Wire Wire Line
+	3150 1300 3700 1300
+Connection ~ 3700 1300
+Wire Wire Line
+	3700 1300 3700 1150
 $EndSCHEMATC

Commit message: uploaded new .stl and BOM
Parts:
- added J12: Conn_01x03_Male, Connector_PinHeader_2.54mm:PinHeader_1x03_P2.54mm_Vertical, symbol Connector:Conn_01x03_Male
Connections:
- wire segments 127 -> 139
Changed lines of the file:
@@
 	1650 2500 1550 2500
 Wire Wire Line
-	1550 2500 1550 2450
-Wire Wire Line
 	1550 2450 1400 2450
 Wire Wire Line
@@
 	1950 1950 2250 1950
 Wire Wire Line
-	2250 1950 2250 2000
-Wire Wire Line
 	1950 2100 2250 2100
 Wire Wire Line
@@
 Wire Wire Line
 	2050 2300 2250 2300
-Wire Wire Line
-	1950 2550 2100 2550
 Wire Wire Line
 	2100 2550 2100 2400
@@
 Wire Wire Line
 	3700 1300 3700 1150
+Wire Wire Line
+	2250 1950 2250 2000
+Wire Wire Line
+	1550 2500 1550 2450
+Wire Wire Line
+	1950 2550 2100 2550
+$Comp
+L Connector:Conn_01x03_Male J12
+U 1 1 5C9CC4B7
+P 1700 1200
+F 0 "J12" V 1760 1340 50  0000 L CNN
+F 1 "Conn_01x03_Male" V 1851 1340 50  0000 L CNN
+F 2 "Connector_PinHeader_2.54mm:PinHeader_1x03_P2.54mm_Vertical" H 1700 1200 50  0001 C CNN
+F 3 "~" H 1700 1200 50  0001 C CNN
+	1    1700 1200
+	0    1    1    0
+$EndComp
+Wire Wire Line
+	2250 1700 2150 1700
+Wire Wire Line
+	2150 1700 2150 1450
+Wire Wire Line
+	2150 1450 1800 1450
+Wire Wire Line
+	1800 1450 1800 1400
+Wire Wire Line
+	2250 1800 2100 1800
+Wire Wire Line
+	2100 1800 2100 1500
+Wire Wire Line
+	2100 1500 1700 1500
+Wire Wire Line
+	1700 1500 1700 1400
+Wire Wire Line
+	2250 1900 2050 1900
+Wire Wire Line
+	2050 1900 2050 1550
+Wire Wire Line
+	2050 1550 1600 1550
+Wire Wire Line
+	1600 1550 1600 1400
 $EndSCHEMATC
